File: Schematics/Proto.sch (EAGLE design)
At the start: 0 parts

Commit message: Some Changes
Changed lines of the file:
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@@
 </sheets>
 </module>
-<module name="PROGRAM-COUNTER" prefix="" dx="30.48" dy="20.32">
+<module name="PROGRAM-COUNTER" prefix="" dx="30.48" dy="50.8">
 <ports>
 <port name="16B_1" side="right" coord="7.62" direction="io"/>
@@
 <port name="|CLR" side="top" coord="0" direction="io"/>
 <port name="GND" side="top" coord="2.54" direction="io"/>
+<port name="CLR" side="top" coord="5.08" direction="io"/>
+<port name="PC_LE" side="top" coord="-12.7" direction="io"/>
+<port name="PC_LRS" side="top" coord="7.62" direction="io"/>
 </ports>
 <variantdefs>
@@
 <segment>
 <label x="63.5" y="205.74" size="1.778" layer="95" rot="R180"/>
+<pinref part="IC4" gate="A" pin="D4"/>
+<wire x1="236.22" y1="172.72" x2="236.22" y2="205.74" width="0.1524" layer="91"/>
 <wire x1="63.5" y1="205.74" x2="93.98" y2="205.74" width="0.1524" layer="91"/>
-</segment>
-<segment>
-<label x="205.74" y="205.74" size="1.778" layer="95" rot="R180"/>
-<wire x1="205.74" y1="205.74" x2="236.22" y2="205.74" width="0.1524" layer="91"/>
-</segment>
-</net>
-<net name="8B_7" class="0">
-<segment>
-<label x="63.5" y="203.2" size="1.778" layer="95" rot="R180"/>
-<wire x1="63.5" y1="203.2" x2="96.52" y2="203.2" width="0.1524" layer="91"/>
-</segment>
-<segment>
-<label x="205.74" y="203.2" size="1.778" layer="95" rot="R180"/>
-<wire x1="205.74" y1="203.2" x2="238.76" y2="203.2" width="0.1524" layer="91"/>
+<wire x1="93.98" y1="205.74" x2="236.22" y2="205.74" width="0.1524" layer="91"/>
+<pinref part="IC2" gate="A" pin="D4"/>
+<wire x1="93.98" y1="172.72" x2="93.98" y2="205.74" width="0.1524" layer="91"/>
 </segment>
 </net>
@@
 <segment>
 <label x="63.5" y="200.66" size="1.778" layer="95" rot="R180"/>
+<pinref part="IC4" gate="A" pin="D2"/>
+<wire x1="241.3" y1="200.66" x2="241.3" y2="172.72" width="0.1524" layer="91"/>
 <wire x1="63.5" y1="200.66" x2="99.06" y2="200.66" width="0.1524" layer="91"/>
-</segment>
-<segment>
-<label x="205.74" y="200.66" size="1.778" layer="95" rot="R180"/>
-<wire x1="205.74" y1="200.66" x2="241.3" y2="200.66" width="0.1524" layer="91"/>
-</segment>
-</net>
-<net name="8B_5" class="0">
-<segment>
-<label x="63.5" y="198.12" size="1.778" layer="95" rot="R180"/>
-<wire x1="63.5" y1="198.12" x2="101.6" y2="198.12" width="0.1524" layer="91"/>
-</segment>
-<segment>
-<label x="205.74" y="198.12" size="1.778" layer="95" rot="R180"/>
-<wire x1="205.74" y1="198.12" x2="243.84" y2="198.12" width="0.1524" layer="91"/>
+<pinref part="IC2" gate="A" pin="D2"/>
+<wire x1="99.06" y1="200.66" x2="241.3" y2="200.66" width="0.1524" layer="91"/>
+<wire x1="99.06" y1="200.66" x2="99.06" y2="172.72" width="0.1524" layer="91"/>
 </segment>
 </net>
@@
 <segment>
 <label x="63.5" y="195.58" size="1.778" layer="95" rot="R180"/>
+<pinref part="IC5" gate="A" pin="D4"/>
+<wire x1="274.32" y1="195.58" x2="274.32" y2="172.72" width="0.1524" layer="91"/>
 <wire x1="63.5" y1="195.58" x2="132.08" y2="195.58" width="0.1524" layer="91"/>
 <pinref part="IC1" gate="A" pin="D4"/>
+<wire x1="132.08" y1="195.58" x2="274.32" y2="195.58" width="0.1524" layer="91"/>
 <wire x1="132.08" y1="195.58" x2="132.08" y2="172.72" width="0.1524" layer="91"/>
 </segment>
-<segment>
-<label x="205.74" y="195.58" size="1.778" layer="95" rot="R180"/>
-<wire x1="205.74" y1="195.58" x2="274.32" y2="195.58" width="0.1524" layer="91"/>
-<pinref part="IC5" gate="A" pin="D4"/>
-<wire x1="274.32" y1="195.58" x2="274.32" y2="172.72" width="0.1524" layer="91"/>
-</segment>
 </net>
 <net name="8B_3" class="0">
 <segment>
+<pinref part="IC5" gate="A" pin="D3"/>
+<wire x1="276.86" y1="193.04" x2="276.86" y2="172.72" width="0.1524" layer="91"/>
 <label x="63.5" y="193.04" size="1.778" layer="95" rot="R180"/>
-<wire x1="63.5" y1="193.04" x2="134.62" y2="193.04" width="0.1524" layer="91"/>
+<wire x1="276.86" y1="193.04" x2="137.16" y2="193.04" width="0.1524" layer="91"/>
 <pinref part="IC1" gate="A" pin="D3"/>
-<wire x1="134.62" y1="187.96" x2="134.62" y2="172.72" width="0.1524" layer="91"/>
-<wire x1="134.62" y1="193.04" x2="134.62" y2="187.96" width="0.1524" layer="91"/>
-</segment>
-<segment>
-<label x="205.74" y="193.04" size="1.778" layer="95" rot="R180"/>
-<wire x1="205.74" y1="193.04" x2="276.86" y2="193.04" width="0.1524" layer="91"/>
-<pinref part="IC5" gate="A" pin="D3"/>
-<wire x1="276.86" y1="187.96" x2="276.86" y2="172.72" width="0.1524" layer="91"/>
-<wire x1="276.86" y1="193.04" x2="276.86" y2="187.96" width="0.1524" layer="91"/>
+<wire x1="134.62" y1="193.04" x2="63.5" y2="193.04" width="0.1524" layer="91"/>
+<wire x1="134.62" y1="172.72" x2="134.62" y2="193.04" width="0.1524" layer="91"/>
+<wire x1="134.62" y1="193.04" x2="137.16" y2="193.04" width="0.1524" layer="91"/>
 </segment>
 </net>
@@
 <segment>
 <label x="63.5" y="190.5" size="1.778" layer="95" rot="R180"/>
+<pinref part="IC5" gate="A" pin="D2"/>
+<wire x1="279.4" y1="190.5" x2="279.4" y2="172.72" width="0.1524" layer="91"/>
 <wire x1="63.5" y1="190.5" x2="137.16" y2="190.5" width="0.1524" layer="91"/>
 <pinref part="IC1" gate="A" pin="D2"/>
+<wire x1="137.16" y1="190.5" x2="279.4" y2="190.5" width="0.1524" layer="91"/>
 <wire x1="137.16" y1="190.5" x2="137.16" y2="172.72" width="0.1524" layer="91"/>
 </segment>
-<segment>
-<label x="205.74" y="190.5" size="1.778" layer="95" rot="R180"/>
-<wire x1="205.74" y1="190.5" x2="279.4" y2="190.5" width="0.1524" layer="91"/>
-<pinref part="IC5" gate="A" pin="D2"/>
-<wire x1="279.4" y1="190.5" x2="279.4" y2="172.72" width="0.1524" layer="91"/>
-</segment>
 </net>
 <net name="8B_1" class="0">
 <segment>
-<label x="63.5" y="187.96" size="1.778" layer="95" rot="R180"/>
-<wire x1="63.5" y1="187.96" x2="109.22" y2="187.96" width="0.1524" layer="91"/>
-<pinref part="IC1" gate="A" pin="D1"/>
-<wire x1="109.22" y1="187.96" x2="111.76" y2="187.96" width="0.1524" layer="91"/>
-<wire x1="139.7" y1="187.96" x2="139.7" y2="172.72" width="0.1524" layer="91"/>
-<wire x1="111.76" y1="187.96" x2="139.7" y2="187.96" width="0.1524" layer="91"/>
-</segment>
-<segment>
-<label x="205.74" y="187.96" size="1.778" layer="95" rot="R180"/>
-<wire x1="205.74" y1="187.96" x2="251.46" y2="187.96" width="0.1524" layer="91"/>
 <pinref part="IC5" gate="A" pin="D1"/>
-<wire x1="251.46" y1="187.96" x2="254" y2="187.96" width="0.1524" layer="91"/>
 <wire x1="281.94" y1="187.96" x2="281.94" y2="172.72" width="0.1524" layer="91"/>
-<wire x1="254" y1="187.96" x2="281.94" y2="187.96" width="0.1524" layer="91"/>
-</segment>
-</net>
-<net name="8B_9" class="0">
-<segment>
-<pinref part="IC2" gate="A" pin="D4"/>
-<wire x1="93.98" y1="172.72" x2="93.98" y2="205.74" width="0.1524" layer="91"/>
-</segment>
-</net>
-<net name="8B_10" class="0">
-<segment>
-<pinref part="IC2" gate="A" pin="D3"/>
-<wire x1="96.52" y1="203.2" x2="96.52" y2="172.72" width="0.1524" layer="91"/>
-</segment>
-</net>
-<net name="8B_11" class="0">
-<segment>
-<pinref part="IC2" gate="A" pin="D2"/>
-<wire x1="99.06" y1="200.66" x2="99.06" y2="172.72" width="0.1524" layer="91"/>
-</segment>
-</net>
-<net name="8B_12" class="0">
-<segment>
-<pinref part="IC2" gate="A" pin="D1"/>
-<wire x1="101.6" y1="198.12" x2="101.6" y2="172.72" width="0.1524" layer="91"/>
+<label x="63.5" y="187.96" size="1.778" layer="95" rot="R180"/>
+<wire x1="281.94" y1="187.96" x2="139.7" y2="187.96" width="0.1524" layer="91"/>
+<pinref part="IC1" gate="A" pin="D1"/>
+<wire x1="139.7" y1="187.96" x2="63.5" y2="187.96" width="0.1524" layer="91"/>
+<wire x1="139.7" y1="172.72" x2="139.7" y2="187.96" width="0.1524" layer="91"/>
 </segment>
 </net>
@@
 </segment>
 </net>
-<net name="8B_13" class="0">
+<net name="8B_5" class="0">
 <segment>
-<pinref part="IC4" gate="A" pin="D4"/>
-<wire x1="236.22" y1="172.72" x2="236.22" y2="205.74" width="0.1524" layer="91"/>
+<pinref part="IC4" gate="A" pin="D1"/>
+<wire x1="243.84" y1="198.12" x2="243.84" y2="172.72" width="0.1524" layer="91"/>
+<label x="63.5" y="198.12" size="1.778" layer="95" rot="R180"/>
+<wire x1="243.84" y1="198.12" x2="104.14" y2="198.12" width="0.1524" layer="91"/>
+<pinref part="IC2" gate="A" pin="D1"/>
+<wire x1="101.6" y1="198.12" x2="63.5" y2="198.12" width="0.1524" layer="91"/>
+<wire x1="101.6" y1="172.72" x2="101.6" y2="198.12" width="0.1524" layer="91"/>
+<wire x1="101.6" y1="198.12" x2="104.14" y2="198.12" width="0.1524" layer="91"/>
 </segment>
 </net>
-<net name="8B_14" class="0">
+<net name="8B_7" class="0">
 <segment>
 <pinref part="IC4" gate="A" pin="D3"/>
 <wire x1="238.76" y1="203.2" x2="238.76" y2="172.72" width="0.1524" layer="91"/>
-</segment>
-</net>
-<net name="8B_15" class="0">
-<segment>
-<pinref part="IC4" gate="A" pin="D2"/>
-<wire x1="241.3" y1="200.66" x2="241.3" y2="172.72" width="0.1524" layer="91"/>
-</segment>
-</net>
-<net name="8B_16" class="0">
-<segment>
-<pinref part="IC4" gate="A" pin="D1"/>
-<wire x1="243.84" y1="198.12" x2="243.84" y2="172.72" width="0.1524" layer="91"/>
+<label x="63.5" y="203.2" size="1.778" layer="95" rot="R180"/>
+<wire x1="238.76" y1="203.2" x2="96.52" y2="203.2" width="0.1524" layer="91"/>
+<pinref part="IC2" gate="A" pin="D3"/>
+<wire x1="96.52" y1="203.2" x2="63.5" y2="203.2" width="0.1524" layer="91"/>
+<wire x1="96.52" y1="203.2" x2="96.52" y2="172.72" width="0.1524" layer="91"/>
 </segment>
 </net>
@@
 <attribute name="NAME" x="-124.46" y="147.32" size="2.032" layer="95" align="bottom-center"/>
 </moduleinst>
-<moduleinst name="PROGRAM-COUNTER1" module="PROGRAM-COUNTER" x="-172.72" y="121.92">
-<attribute name="NAME" x="-172.72" y="121.92" size="2.032" layer="95" align="bottom-center"/>
-</moduleinst>
 <moduleinst name="RAM1" module="RAM" x="-119.38" y="114.3">
 <attribute name="NAME" x="-119.38" y="114.3" size="2.032" layer="95" align="bottom-center"/>
 </moduleinst>
+<moduleinst name="PROGRAM-COUNTER1" module="PROGRAM-COUNTER" x="-182.88" y="104.14">
+<attribute name="NAME" x="-182.88" y="104.14" size="2.032" layer="95" align="bottom-center"/>
+</moduleinst>
 </moduleinsts>

Commit message: PCB Design Started
Parts:
- added LED1, LED2, LED3, LED4, LED5, LED6, LED7, LED8: (no value), led:LED5MM
- added R1, R2, R3, R4, R5, R6, R7, R8: 10k, rcl:R-EU_0204/7
- added X1: (no value), con-wago-500:W237-102
Connections:
- new net 8B_1: LED1.A, R1.2
- new net 8B_2: LED2.A, R2.2
- new net 8B_3: LED3.A, R3.2
- new net 8B_4: LED4.A, R4.2
- new net 8B_5: LED5.A, R8.1
- new net 8B_6: LED6.A, R7.1
- new net 8B_7: LED7.A, R6.1
- new net 8B_8: LED8.A, R5.1
- new net ALUSUB: LED3.A
- new net CLK: LED1.A
- new net GND: LED1.C, LED2.C, LED3.C, LED4.C, LED5.C, LED6.C, LED7.C, LED8.C, R1.1, R2.1, R3.1, R4.1, R5.2, R6.2, R7.2, R8.2, X1-2.KL
- new net N$1: R5.1
- new net N$11: R2.1, R7.S
- new net N$17: LED1.A
- new net N$18: LED2.A
- new net N$19: LED3.A
- new net N$2: R3.1
- new net N$20: LED4.A
- new net N$25: LED5.A
- new net N$26: LED6.A
- new net N$27: LED6.A, LED7.A
- new net N$28: LED8.A
- new net N$3: R6.1
- new net N$7: R4.1
- new net N$9: R1.1, R2.2
- new net NNOW: LED7.A
- new net NNOW2: LED8.A
- new net PC_LE: LED2.A
- new net PC_LRS: LED1.A
- new net TRIGGER: R7.E
- new net VCC: R1.2, R3.2, R4.2, R5.2, R6.2, X1-1.KL
- new net |ALUWRITE: LED4.A
- new net |FL: LED5.A

Commit message: PCB Made Better
Parts:
- removed LED1, LED2, LED3, LED4, LED5, LED6, LED7, LED8: (no value), led:LED5MM
- removed R1, R2, R3, R4, R5, R6, R7: 10k, rcl:R-EU_0204/7
- added 1, 11, 12, 13, 2, 3, 5: 10k, rcl:R-EU_0204/7
- added C1: 330uf, rcl:C-EU025-025X050
- added L1, L2, L3, L4, L5, L6, L7, L8: (no value), led:LED5MM
- added R10, R11, R12, R13, R14, R15, R16, R9: 220, rcl:R-EU_0204/7
- renumbered R8 to 15
Connections:
- removed net ALUSUB: LED3.A
- removed net CLK: LED1.A
- removed net N$11: R2.1, R7.S
- removed net N$20: LED4.A
- removed net N$25: LED5.A
- removed net N$26: LED6.A
- removed net N$27: LED6.A, LED7.A
- removed net N$28: LED8.A
- removed net NNOW: LED7.A
- removed net NNOW2: LED8.A
- removed net PC_LE: LED2.A
- removed net PC_LRS: LED1.A
- removed net |ALUWRITE: LED4.A
- removed net |FL: LED5.A
- new net N$100: R14.2
- new net N$101: R15.2
- new net N$102: R16.2
- new net N$12: R9.2
- new net N$13: R10.2
- new net N$14: R11.2
- new net N$15: R12.2
- new net N$16: R13.2
- new net N$38: L1.C, R9.2
- new net N$39: L2.C, R10.2
- new net N$40: L3.C, R11.2
- new net N$41: L4.C, R12.2
- new net N$42: L5.C, R13.2
- new net N$43: L6.C, R14.2
- new net N$44: L7.C, R15.2
- new net N$45: L8.C, R16.2, R9.2
- new net N$46: R10.2
- new net N$47: R11.2
- new net N$48: R12.2
- new net N$49: R13.2
- new net N$5: R12.2
- new net N$50: R14.2
- new net N$51: R15.2
- new net N$52: R16.2
- new net N$6: R13.2
- new net N$8: R15.2
- new net N$95: R9.2
- new net N$96: R10.2
- new net N$97: R11.2
- new net N$98: R12.2
- new net N$99: R13.2
- net 8B_1: now also 1.2, L1.A; no longer LED1.A, R1.2
- net 8B_2: now also 2.2, L2.A; no longer LED2.A, R2.2
- net 8B_3: now also 3.2, L3.A; no longer LED3.A, R3.2
- net 8B_4: now also 5.2, L4.A; no longer LED4.A, R4.2
- net 8B_5: now also L5.A; no longer LED5.A
- net 8B_6: now also 13.1, L6.A; no longer LED6.A, R7.1
- net 8B_7: now also 12.1, L7.A; no longer LED7.A, R6.1
- net 8B_8: now also 11.1, L8.A; no longer LED8.A, R5.1
- net GND: now also 1.1, 11.2, 12.2, 13.2, 2.1, 3.1, 5.1, C1.2, R10.1, R11.1, R12.1, R13.1, R14.1, R15.1, R16.1, R9.1; no longer LED1.C, LED2.C, LED3.C, LED4.C, LED5.C, LED6.C, LED7.C, LED8.C, R1.1, R2.1, R3.1, R4.1, R5.2, R6.2, R7.2
- net N$1: now also R9.2; no longer R5.1
- net N$17: now also R14.2; no longer LED1.A
- net N$18: now also R15.2; no longer LED2.A
- net N$19: now also R16.2; no longer LED3.A
- net N$2: now also R10.2; no longer R3.1
- net N$3: now also R11.2; no longer R6.1
- net N$7: now also R14.2; no longer R4.1
- net N$9: now also R16.2; no longer R1.1, R2.2
- net TRIGGER: now also C1.1; no longer R7.E
- net VCC: now also C1.1; no longer R1.2, R3.2, R4.2, R5.2, R6.2
