File: Schematics/proto.brd (EAGLE design)
At the start: 525.8 x 437.8 mm, 168 parts

Commit message: Organized
Parts:
- moved CONTROL_LOGIC1:LED14 80.9 mm to (174.0, -47.0)
- moved CONTROL_LOGIC1:LED21 80.9 mm to (174.0, -38.1)
- moved CONTROL_LOGIC1:LED6 80.9 mm to (174.0, -29.2)
- moved CONTROL_LOGIC1:LED1 80.9 mm to (114.3, -38.1)
- moved CONTROL_LOGIC1:LED10 80.9 mm to (58.4, -29.2)
- moved CONTROL_LOGIC1:LED11 80.9 mm to (143.5, -38.1)
- moved CONTROL_LOGIC1:LED12 80.9 mm to (29.2, -29.2)
- moved CONTROL_LOGIC1:LED13 80.9 mm to (204.5, -47.0)
- moved CONTROL_LOGIC1:LED15 80.9 mm to (143.5, -47.0)
- moved CONTROL_LOGIC1:LED16 80.9 mm to (114.3, -47.0)
- moved CONTROL_LOGIC1:LED17 80.9 mm to (85.1, -47.0)
- moved CONTROL_LOGIC1:LED18 80.9 mm to (58.4, -47.0)
- moved CONTROL_LOGIC1:LED19 80.9 mm to (29.2, -47.0)
- moved CONTROL_LOGIC1:LED2 80.9 mm to (85.1, -38.1)
- moved CONTROL_LOGIC1:LED20 80.9 mm to (204.5, -38.1)
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Routing:
- net 8B_2: track 0.00 -> 397.5 mm
- net 8B_1: track 0.00 -> 397.5 mm
- net 8B_8: track 0.00 -> 396.2 mm
- net 8B_7: track 0.00 -> 396.2 mm
- net 8B_6: track 0.00 -> 396.2 mm
- net 8B_5: track 0.00 -> 396.2 mm
- net 8B_4: track 0.00 -> 396.2 mm
- net 8B_3: track 0.00 -> 396.2 mm
Other:
- board size 525.8 x 437.8 mm -> 535.9 x 575 mm

Commit message: PCB Made Better
Parts:
- removed R1, R2, R3, R4, R5, R6, R7, R8: 10k, rcl:0204/7
- removed RAM1:M_ADDR: 1-794681-6, con-amp:1-794681-6
- added 1, 11, 12, 13, 15, 2, 3, 5: 10k, rcl:0204/7
- added C1: 330uf, rcl:C025-025X050
- added CLK1:R13, CONTROL_LOGIC1:R1, CONTROL_LOGIC1:R10, CONTROL_LOGIC1:R11, CONTROL_LOGIC1:R12, CONTROL_LOGIC1:R13, CONTROL_LOGIC1:R14, CONTROL_LOGIC1:R15, CONTROL_LOGIC1:R16, CONTROL_LOGIC1:R17, CONTROL_LOGIC1:R18, CONTROL_LOGIC1:R19, CONTROL_LOGIC1:R2, CONTROL_LOGIC1:R20, CONTROL_LOGIC1:R21, CONTROL_LOGIC1:R3, CONTROL_LOGIC1:R4, CONTROL_LOGIC1:R5, CONTROL_LOGIC1:R6, CONTROL_LOGIC1:R7, CONTROL_LOGIC1:R8, CONTROL_LOGIC1:R9, INST_REGISTER1:R10, INST_REGISTER1:R11, INST_REGISTER1:R12, INST_REGISTER1:R13, INST_REGISTER1:R14, INST_REGISTER1:R15, INST_REGISTER1:R16, INST_REGISTER1:R9, PROGRAM-COUNTER1:R1, PROGRAM-COUNTER1:R10, PROGRAM-COUNTER1:R11, PROGRAM-COUNTER1:R12, PROGRAM-COUNTER1:R13, PROGRAM-COUNTER1:R14, PROGRAM-COUNTER1:R15, PROGRAM-COUNTER1:R16, PROGRAM-COUNTER1:R2, PROGRAM-COUNTER1:R3, PROGRAM-COUNTER1:R4, PROGRAM-COUNTER1:R5, PROGRAM-COUNTER1:R6, PROGRAM-COUNTER1:R7, PROGRAM-COUNTER1:R8, PROGRAM-COUNTER1:R9, R10, R11, R12, R13, R14, R15, R16, R9, RAM1:R10, RAM1:R11, RAM1:R12, RAM1:R13, RAM1:R14, RAM1:R15, RAM1:R16, RAM1:R9: 220, rcl:0204/7
- added RAM1:JP1, RAM1:JP10, RAM1:JP11, RAM1:JP12, RAM1:JP13, RAM1:JP14, RAM1:JP15, RAM1:JP16, RAM1:JP2, RAM1:JP3, RAM1:JP4, RAM1:JP5, RAM1:JP6, RAM1:JP7, RAM1:JP8, RAM1:JP9: (no value), pinhead:1X01
- moved INST_REGISTER1:IC3 176.6 mm to (117.1, 281.2), turned to 0 degrees
- moved INST_REGISTER1:LED16 171.1 mm to (141.0, 238.0), turned to 0 degrees
- moved INST_REGISTER1:LED15 164.4 mm to (134.6, 238.0), turned to 0 degrees
- moved INST_REGISTER1:LED14 158.0 mm to (128.3, 238.0), turned to 0 degrees
- moved INST_REGISTER1:LED13 151.8 mm to (121.9, 238.0), turned to 0 degrees
- moved CONTROL_LOGIC1:IC2 149.6 mm to (150.6, 170.9), turned to 180 degrees
- moved CONTROL_LOGIC1:IC1 148.5 mm to (114.8, 170.9), turned to 180 degrees
- moved INST_REGISTER1:LED12 146.0 mm to (115.6, 238.0), turned to 0 degrees
- moved ALU1:IC4 145.5 mm to (357.1, 217.9), turned to 270 degrees
- moved INST_REGISTER1:LED11 140.4 mm to (109.2, 238.0), turned to 0 degrees
- moved INST_REGISTER1:LED10 135.2 mm to (102.9, 238.0), turned to 0 degrees
- moved ALU1:V1 132.4 mm to (381.3, 217.7), turned to 90 degrees
- moved ALU1:V2 132.2 mm to (396.7, 217.4), turned to 90 degrees
- moved INST_REGISTER1:IC4 130.8 mm to (128.3, 207.5), turned to 0 degrees
- moved INST_REGISTER1:LED9 130.5 mm to (96.5, 238.0), turned to 0 degrees
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- renumbered LED1 to L1, LED2 to L2, LED3 to L3, LED4 to L4, LED5 to L5, LED6 to L6, LED7 to L7, LED8 to L8
Connections:
- new net CLK1:N$6: CLK1:LED1.K, CLK1:R13.2
- new net CONTROL_LOGIC1:N$12: CONTROL_LOGIC1:LED6.K, CONTROL_LOGIC1:R9.2
- new net CONTROL_LOGIC1:N$13: CONTROL_LOGIC1:LED7.K, CONTROL_LOGIC1:R10.2
- new net CONTROL_LOGIC1:N$14: CONTROL_LOGIC1:LED8.K, CONTROL_LOGIC1:R11.2
- new net CONTROL_LOGIC1:N$15: CONTROL_LOGIC1:LED17.K, CONTROL_LOGIC1:R12.2
- new net CONTROL_LOGIC1:N$16: CONTROL_LOGIC1:LED18.K, CONTROL_LOGIC1:R13.2
- new net CONTROL_LOGIC1:N$17: CONTROL_LOGIC1:LED19.K, CONTROL_LOGIC1:R14.2
- new net CONTROL_LOGIC1:N$18: CONTROL_LOGIC1:LED20.K, CONTROL_LOGIC1:R15.2
- new net CONTROL_LOGIC1:N$19: CONTROL_LOGIC1:LED21.K, CONTROL_LOGIC1:R16.2
- new net CONTROL_LOGIC1:N$20: CONTROL_LOGIC1:LED1.K, CONTROL_LOGIC1:R1.2
- new net CONTROL_LOGIC1:N$21: CONTROL_LOGIC1:LED2.K, CONTROL_LOGIC1:R2.2
- new net CONTROL_LOGIC1:N$22: CONTROL_LOGIC1:LED3.K, CONTROL_LOGIC1:R3.2
- new net CONTROL_LOGIC1:N$23: CONTROL_LOGIC1:LED4.K, CONTROL_LOGIC1:R4.2
- new net CONTROL_LOGIC1:N$24: CONTROL_LOGIC1:LED5.K, CONTROL_LOGIC1:R5.2
- new net CONTROL_LOGIC1:N$25: CONTROL_LOGIC1:LED14.K, CONTROL_LOGIC1:R6.2
- new net CONTROL_LOGIC1:N$26: CONTROL_LOGIC1:LED15.K, CONTROL_LOGIC1:R7.2
- new net CONTROL_LOGIC1:N$28: CONTROL_LOGIC1:LED16.K, CONTROL_LOGIC1:R8.2
- new net CONTROL_LOGIC1:N$29: CONTROL_LOGIC1:LED9.K, CONTROL_LOGIC1:R17.2
- new net CONTROL_LOGIC1:N$30: CONTROL_LOGIC1:LED10.K, CONTROL_LOGIC1:R18.2
- new net CONTROL_LOGIC1:N$31: CONTROL_LOGIC1:LED11.K, CONTROL_LOGIC1:R19.2
- new net CONTROL_LOGIC1:N$32: CONTROL_LOGIC1:LED12.K, CONTROL_LOGIC1:R20.2
- new net CONTROL_LOGIC1:N$33: CONTROL_LOGIC1:LED13.K, CONTROL_LOGIC1:R21.2
- new net INST_REGISTER1:N$1: INST_REGISTER1:LED9.K, INST_REGISTER1:R9.2
- new net INST_REGISTER1:N$2: INST_REGISTER1:LED10.K, INST_REGISTER1:R10.2
- new net INST_REGISTER1:N$3: INST_REGISTER1:LED11.K, INST_REGISTER1:R11.2
- new net INST_REGISTER1:N$5: INST_REGISTER1:LED12.K, INST_REGISTER1:R12.2
- new net INST_REGISTER1:N$6: INST_REGISTER1:LED13.K, INST_REGISTER1:R13.2
- new net INST_REGISTER1:N$7: INST_REGISTER1:LED14.K, INST_REGISTER1:R14.2
- new net INST_REGISTER1:N$8: INST_REGISTER1:LED15.K, INST_REGISTER1:R15.2
- new net INST_REGISTER1:N$9: INST_REGISTER1:LED16.K, INST_REGISTER1:R16.2
- new net N$38: L1.K, R9.2
- new net N$39: L2.K, R10.2
- new net N$40: L3.K, R11.2
- new net N$41: L4.K, R12.2
- new net N$42: L5.K, R13.2
- new net N$43: L6.K, R14.2
- new net N$44: L7.K, R15.2
- new net N$45: L8.K, R16.2
- new net PROGRAM-COUNTER1:N$45: PROGRAM-COUNTER1:LED9.K, PROGRAM-COUNTER1:R9.2
- new net PROGRAM-COUNTER1:N$46: PROGRAM-COUNTER1:LED10.K, PROGRAM-COUNTER1:R10.2
- new net PROGRAM-COUNTER1:N$47: PROGRAM-COUNTER1:LED11.K, PROGRAM-COUNTER1:R11.2
- new net PROGRAM-COUNTER1:N$48: PROGRAM-COUNTER1:LED12.K, PROGRAM-COUNTER1:R12.2
- new net PROGRAM-COUNTER1:N$49: PROGRAM-COUNTER1:LED13.K, PROGRAM-COUNTER1:R13.2
- new net PROGRAM-COUNTER1:N$50: PROGRAM-COUNTER1:LED14.K, PROGRAM-COUNTER1:R14.2
- new net PROGRAM-COUNTER1:N$51: PROGRAM-COUNTER1:LED15.K, PROGRAM-COUNTER1:R15.2
- new net PROGRAM-COUNTER1:N$52: PROGRAM-COUNTER1:LED16.K, PROGRAM-COUNTER1:R16.2
- new net PROGRAM-COUNTER1:N$53: PROGRAM-COUNTER1:LED1.K, PROGRAM-COUNTER1:R1.2
- new net PROGRAM-COUNTER1:N$54: PROGRAM-COUNTER1:LED2.K, PROGRAM-COUNTER1:R2.2
- new net PROGRAM-COUNTER1:N$55: PROGRAM-COUNTER1:LED3.K, PROGRAM-COUNTER1:R3.2
- new net PROGRAM-COUNTER1:N$56: PROGRAM-COUNTER1:LED4.K, PROGRAM-COUNTER1:R4.2
- new net PROGRAM-COUNTER1:N$57: PROGRAM-COUNTER1:LED5.K, PROGRAM-COUNTER1:R5.2
- new net PROGRAM-COUNTER1:N$58: PROGRAM-COUNTER1:LED6.K, PROGRAM-COUNTER1:R6.2
- new net PROGRAM-COUNTER1:N$59: PROGRAM-COUNTER1:LED7.K, PROGRAM-COUNTER1:R7.2
- new net PROGRAM-COUNTER1:N$60: PROGRAM-COUNTER1:LED8.K, PROGRAM-COUNTER1:R8.2
- new net RAM1:N$100: RAM1:LED14.K, RAM1:R14.2
- new net RAM1:N$101: RAM1:LED15.K, RAM1:R15.2
- new net RAM1:N$102: RAM1:LED16.K, RAM1:R16.2
- new net RAM1:N$95: RAM1:LED9.K, RAM1:R9.2
- new net RAM1:N$96: RAM1:LED10.K, RAM1:R10.2
- new net RAM1:N$97: RAM1:LED11.K, RAM1:R11.2
- new net RAM1:N$98: RAM1:LED12.K, RAM1:R12.2
- new net RAM1:N$99: RAM1:LED13.K, RAM1:R13.2
- net 8B_1: now also 1.2; no longer R1.2
- net 8B_2: now also 2.2; no longer R2.2
- net 8B_3: now also 3.2; no longer R3.2
- net 8B_4: now also 5.2; no longer R4.2
- net 8B_5: now also 15.1; no longer R8.1
- net 8B_6: now also 13.1; no longer R7.1
- net 8B_7: now also 12.1; no longer R6.1
- net 8B_8: now also 11.1; no longer R5.1
- net GND: now also 1.1, 11.2, 12.2, 13.2, 15.2, 2.1, 3.1, 5.1, C1.2, CLK1:R13.1, CONTROL_LOGIC1:R1.1, CONTROL_LOGIC1:R10.1, CONTROL_LOGIC1:R11.1, CONTROL_LOGIC1:R12.1, CONTROL_LOGIC1:R13.1, CONTROL_LOGIC1:R14.1, CONTROL_LOGIC1:R15.1, CONTROL_LOGIC1:R16.1, CONTROL_LOGIC1:R17.1, CONTROL_LOGIC1:R18.1, CONTROL_LOGIC1:R19.1, CONTROL_LOGIC1:R2.1, CONTROL_LOGIC1:R20.1, CONTROL_LOGIC1:R21.1, CONTROL_LOGIC1:R3.1, CONTROL_LOGIC1:R4.1, CONTROL_LOGIC1:R5.1, CONTROL_LOGIC1:R6.1, CONTROL_LOGIC1:R7.1, CONTROL_LOGIC1:R8.1, CONTROL_LOGIC1:R9.1, INST_REGISTER1:R10.1, INST_REGISTER1:R11.1, INST_REGISTER1:R12.1, INST_REGISTER1:R13.1, INST_REGISTER1:R14.1, INST_REGISTER1:R15.1, INST_REGISTER1:R16.1, INST_REGISTER1:R9.1, PROGRAM-COUNTER1:R1.1, PROGRAM-COUNTER1:R10.1, PROGRAM-COUNTER1:R11.1, PROGRAM-COUNTER1:R12.1, PROGRAM-COUNTER1:R13.1, PROGRAM-COUNTER1:R14.1, PROGRAM-COUNTER1:R15.1, PROGRAM-COUNTER1:R16.1, PROGRAM-COUNTER1:R2.1, PROGRAM-COUNTER1:R3.1, PROGRAM-COUNTER1:R4.1, PROGRAM-COUNTER1:R5.1, PROGRAM-COUNTER1:R6.1, PROGRAM-COUNTER1:R7.1, PROGRAM-COUNTER1:R8.1, PROGRAM-COUNTER1:R9.1, R10.1, R11.1, R12.1, R13.1, R14.1, R15.1, R16.1, R9.1; no longer CLK1:LED1.K, CONTROL_LOGIC1:LED1.K, CONTROL_LOGIC1:LED10.K, CONTROL_LOGIC1:LED11.K, CONTROL_LOGIC1:LED12.K, CONTROL_LOGIC1:LED13.K, CONTROL_LOGIC1:LED14.K, CONTROL_LOGIC1:LED15.K, CONTROL_LOGIC1:LED16.K, CONTROL_LOGIC1:LED17.K, CONTROL_LOGIC1:LED18.K, CONTROL_LOGIC1:LED19.K, CONTROL_LOGIC1:LED2.K, CONTROL_LOGIC1:LED20.K, CONTROL_LOGIC1:LED21.K, CONTROL_LOGIC1:LED3.K, CONTROL_LOGIC1:LED4.K, CONTROL_LOGIC1:LED5.K, CONTROL_LOGIC1:LED6.K, CONTROL_LOGIC1:LED7.K, CONTROL_LOGIC1:LED8.K, CONTROL_LOGIC1:LED9.K, INST_REGISTER1:LED10.K, INST_REGISTER1:LED11.K, INST_REGISTER1:LED12.K, INST_REGISTER1:LED13.K, INST_REGISTER1:LED14.K, INST_REGISTER1:LED15.K, INST_REGISTER1:LED16.K, INST_REGISTER1:LED9.K, L1.K, L2.K, L3.K, L4.K, L5.K, L6.K, L7.K, L8.K, PROGRAM-COUNTER1:LED1.K, PROGRAM-COUNTER1:LED10.K, PROGRAM-COUNTER1:LED11.K, PROGRAM-COUNTER1:LED12.K, PROGRAM-COUNTER1:LED13.K, PROGRAM-COUNTER1:LED14.K, PROGRAM-COUNTER1:LED15.K, PROGRAM-COUNTER1:LED16.K, PROGRAM-COUNTER1:LED2.K, PROGRAM-COUNTER1:LED3.K, PROGRAM-COUNTER1:LED4.K, PROGRAM-COUNTER1:LED5.K, PROGRAM-COUNTER1:LED6.K, PROGRAM-COUNTER1:LED7.K, PROGRAM-COUNTER1:LED8.K, PROGRAM-COUNTER1:LED9.K, R1.1, R2.1, R3.1, R4.1, R5.2, R6.2, R7.2, R8.2
- net RAM1:GND: now also RAM1:R10.1, RAM1:R11.1, RAM1:R12.1, RAM1:R13.1, RAM1:R14.1, RAM1:R15.1, RAM1:R16.1, RAM1:R9.1; no longer RAM1:LED10.K, RAM1:LED11.K, RAM1:LED12.K, RAM1:LED13.K, RAM1:LED14.K, RAM1:LED15.K, RAM1:LED16.K, RAM1:LED9.K
- net RAM1:N$20: now also RAM1:JP1.1; no longer RAM1:M_ADDR.1
- net RAM1:N$21: now also RAM1:JP2.1; no longer RAM1:M_ADDR.3
- net RAM1:N$22: now also RAM1:JP3.1; no longer RAM1:M_ADDR.5
- net RAM1:N$23: now also RAM1:JP4.1; no longer RAM1:M_ADDR.7
- net RAM1:N$24: now also RAM1:JP5.1; no longer RAM1:M_ADDR.9
- net RAM1:N$25: now also RAM1:JP6.1; no longer RAM1:M_ADDR.11
- net RAM1:N$26: now also RAM1:JP7.1; no longer RAM1:M_ADDR.13
- net RAM1:N$27: now also RAM1:JP8.1; no longer RAM1:M_ADDR.15
- net RAM1:N$28: now also RAM1:JP13.1; no longer RAM1:M_ADDR.2
- net RAM1:N$29: now also RAM1:JP14.1; no longer RAM1:M_ADDR.4
- net RAM1:N$30: now also RAM1:JP15.1; no longer RAM1:M_ADDR.6
- net RAM1:N$31: now also RAM1:JP16.1; no longer RAM1:M_ADDR.8
- net RAM1:N$32: now also RAM1:JP9.1; no longer RAM1:M_ADDR.10
- net RAM1:N$33: now also RAM1:JP10.1; no longer RAM1:M_ADDR.12
- net RAM1:N$34: now also RAM1:JP11.1; no longer RAM1:M_ADDR.14
- net RAM1:N$35: now also RAM1:JP12.1; no longer RAM1:M_ADDR.16
- net RAM1:N$53: now also RAM1:IC15.3
- net RAM1:N$87: now also RAM1:IC17.3
- net VCC: now also C1.1
Routing:
- net 8B_2: track 397.5 -> 247.9 mm
- net 8B_1: track 397.5 -> 247.9 mm
- net 8B_8: track 396.2 -> 246.6 mm
- net 8B_7: track 396.2 -> 246.6 mm
- net 8B_6: track 396.2 -> 246.6 mm
- net 8B_5: track 396.2 -> 246.6 mm
- net 8B_4: track 396.2 -> 246.6 mm
- net 8B_3: track 396.2 -> 246.6 mm
Other:
- board size 535.9 x 575 mm -> 536.4 x 400 mm

Commit message: Board Edited
Parts:
- moved 11 82.5 mm to (213.9, 354.1), turned to 90 degrees
- moved 12 77.9 mm to (218.9, 354.1), turned to 90 degrees
- moved 1 77.3 mm to (249.4, 354.1), turned to 270 degrees
- moved 13 74.4 mm to (224.0, 354.1), turned to 90 degrees
- moved 2 74.0 mm to (244.3, 354.1), turned to 270 degrees
- moved 15 72.2 mm to (229.1, 354.1), turned to 90 degrees
- moved 3 72.0 mm to (239.3, 354.1), turned to 270 degrees
- moved 5 71.4 mm to (234.2, 354.1), turned to 270 degrees
- moved ALU1:IC8 65.5 mm to (327.9, 80.0), turned to 270 degrees
- moved R16 63.8 mm to (213.9, 365.5), turned to 90 degrees
- moved L8 62.7 mm to (205.0, 379.5), turned to 270 degrees
- moved R15 57.7 mm to (218.9, 365.5), turned to 90 degrees
- moved B_REGISTER1:IC8 57.0 mm to (327.2, 142.2)
- moved R9 56.9 mm to (249.4, 365.5), turned to 90 degrees
- moved B_REGISTER1:IC7 53.0 mm to (327.9, 116.1), turned to 270 degrees
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Routing:
- net 8B_1: track 247.9 -> 0.72 mm
- net 8B_2: track 247.9 -> 0.72 mm
- net 8B_6: track 246.6 -> 0.72 mm
- net 8B_5: track 246.6 -> 0.72 mm
- net 8B_8: track 246.6 -> 0.72 mm
- net 8B_7: track 246.6 -> 0.72 mm
- net 8B_4: track 246.6 -> 0.72 mm
- net 8B_3: track 246.6 -> 0.72 mm
- added copper zone on layer 1, net GND
- added copper zone on layer 16, net GND
Other:
- board size 536.4 x 400 mm -> 478.3 x 402 mm
- board text added: "A Register/A Kaydedicisi"
- board text added: "ALU/Mantıksal İşlem Birimi"
- board text added: "B Register/B Kaydedicisi"
- board text added: "Clock/Saat"
- board text added: "Control Logic/Kontrol Mantığı"
- board text added: "Controll Signals/Kontrol Sinyalleri"
- board text added: "Instruction Register/Talimat Kaydedicisi"
- board text added: "Program Counter/Program Sayıcı"

Commit message: Small Fix
Other:
- board size 478.3 x 402 mm -> 482.6 x 402 mm
Changed lines of the file:
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@@
 <fusionsync huburn="a.cGVyc29uYWw6dWUyYzAxZDJj" projecturn="a.cGVyc29uYWw6dWUyYzAxZDJjIzIwMTkwNTA1MTkyMDg5NTI2" f3durn="urn:adsk.wipprod:dm.lineage:70GWcDjMSPOcQDQjk4DCcg" pcbguid="22574776-4e41-4d66-91ec-4a67a1a4bc81" lastpulledtime="" lastsyncedchangeguid="bd499cde-6b20-ed0b-bac9-61ddcb5f395d"/>
 <plain>
-<wire x1="-15.494" y1="38.354" x2="459.72" y2="40.386" width="0" layer="20"/>
-<wire x1="459.72" y1="40.386" x2="459.212" y2="440.36" width="0" layer="20"/>
-<wire x1="459.212" y1="440.36" x2="-18.542" y2="438.328" width="0" layer="20"/>
-<wire x1="-18.542" y1="438.328" x2="-15.494" y2="38.354" width="0" layer="20"/>
+<wire x1="-23.368" y1="39.37" x2="459.212" y2="38.862" width="0" layer="20"/>
+<wire x1="459.212" y1="38.862" x2="459.212" y2="440.36" width="0" layer="20"/>
+<wire x1="459.212" y1="440.36" x2="-23.368" y2="440.868" width="0" layer="20"/>
+<wire x1="-23.368" y1="440.868" x2="-23.368" y2="39.37" width="0" layer="20"/>
 <text x="53.086" y="377.952" size="1.778" layer="21">Clock/Saat</text>
 <text x="371.094" y="268.732" size="1.778" layer="21">Program Counter/Program Sayıcı</text>

Commit message: Added renderings and autoroute schematics
Routing:
- net VCC: track 0.00 -> 1132.9 mm, vias 0 -> 5
- net CLK: track 0.00 -> 1071.1 mm, vias 0 -> 3
- net RAM1:GND: track 0.00 -> 753.9 mm
- net 8B_2: track 0.72 -> 714.9 mm, vias 0 -> 12
- net 8B_1: track 0.72 -> 714.2 mm, vias 0 -> 10
- net CLR: track 0.00 -> 696.5 mm, vias 0 -> 6
- net 8B_3: track 0.72 -> 674.2 mm, vias 0 -> 9
- net 8B_4: track 0.72 -> 652.2 mm, vias 0 -> 9
- net 8B_6: track 0.72 -> 623.3 mm, vias 0 -> 3
- net 8B_8: track 0.72 -> 599.2 mm, vias 0 -> 4
- net 8B_5: track 0.72 -> 592.0 mm, vias 0 -> 6
- net 8B_7: track 0.72 -> 591.7 mm, vias 0 -> 2
- net COUNT: track 0.00 -> 531.6 mm, vias 0 -> 8
- net PC_LE: track 0.00 -> 522.2 mm, vias 0 -> 5
- net RAM1:VCC: track 0.00 -> 518.8 mm, vias 0 -> 3
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