File: Schematics/GPU/GPU.sch (EAGLE design)
At the start: 4 parts

Commit message: Routd and Cams Created
Parts:
- added C2: 1n, resistor:C-EU025-025X050
- added IC2: 74ACT04N, 74xx-eu:74ACT04N
- added IC3: 74ACT30N, 74xx-eu:74ACT30N
- added IC4: 74AC151N, 74xx-eu:74AC151N
- added JP4: (no value), pinhead:PINHD-1X2
- added Q1: (no value), special:XTAL/S
- added R1, R2: 220, rcl:R-EU_0204/7
- added V1, V2: 74161N, 74ttl-din:74161N
- added V3: 744040N, 74ttl-din:744040N
- added V4: 7420N, 74ttl-din:7420N
Connections:
- new net GND: IC1.VSS, JP4.1, V11.A, V11.B, V11.C, V11.D, V21.A, V21.B, V21.C, V21.D, V31.CLR
- new net HSYNC: V4/1.Y
- new net N$1: IC2D.I, Q1.2, R1.1
- new net N$10: IC1.A4, V31.QE, V4/1.A
- new net N$11: IC1.A6, V31.QG, V4/1.C, V4/1.D
- new net N$12: IC1.A11, IC3A.I4, V21.CLK, V31.QL
- new net N$13: IC1.A7, IC3A.I7, V31.QH
- new net N$14: V21.!LOAD, V4/2.Y
- new net N$15: IC1.A14, V21.QC, V4/2.A
- new net N$16: IC3A.I1, V21.QD, V4/2.B, V4/2.C, V4/2.D
- new net N$17: IC1.A8, IC3A.I6, V31.QI
- new net N$18: IC1.A9, IC3A.I5, V31.QJ
- new net N$19: IC1.A12, IC3A.I3, V21.QA
- new net N$2: C2.2, IC2D.O, R1.2
- new net N$20: IC1.A13, IC3A.I2, V21.QB
- new net N$21: IC1.A5, IC2C.I, V31.QK
- new net N$22: IC2C.O, IC3A.I0
- new net N$23: IC2F.I, IC3A.O
- new net N$24: IC4A.A, V11.QA
- new net N$25: IC4A.B, V11.QB
- new net N$26: IC4A.G, V11.QD
- new net N$27: IC1.I/O0, IC4A.D0
- new net N$28: IC1.I/O1, IC4A.D1
- new net N$29: IC1.I/O2, IC4A.D2
- new net N$3: C2.1, IC2E.I, R2.1
- new net N$30: IC1.I/O3, IC4A.D3
- new net N$31: IC1.I/O4, IC4A.D4
- new net N$32: IC1.I/O5, IC4A.D5
- new net N$33: IC1.I/O6, IC4A.D6
- new net N$34: IC1.I/O7, IC4A.D7
- new net N$35: IC1.A0, V31.QA
- new net N$36: IC1.A1, V31.QB
- new net N$37: IC1.A2, V31.QC
- new net N$38: IC1.A3, V31.QD
- new net N$39: IC2B.O, V4/1.B
- new net N$4: IC2E.O, Q1.1, R2.2, V11.CLK
- new net N$44: IC1.A10, IC2B.I, V31.QF
- new net N$5: IC2A.O, V11.!LOAD
- new net N$6: IC4A.C, V11.QC, V31.CLK
- new net N$7: IC2A.I, V11.RCO
- new net VCC: IC1.VCC, JP4.2, V11.!CLR, V21.!CLR
- new net VSYNC: IC2F.O
Other:
- moved on the sheet: IC1, JP1, JP2, JP3

Commit message: Design İmproved
Parts:
- removed JP3: (no value), pinhead:PINHD-1X1
- added IC10: 74AC04N, 74xx-eu:74AC04N
- added IC5, IC6, IC7, IC8, IC9: 74AC245N, 74xx-eu:74AC245N
- added J1: (no value), Wurth_Elektronik_Electromechanic_Input-Output_Connectors_rev19a:618015325223
- added JP5: (no value), pinhead:PINHD-1X1
- added JP6: (no value), pinhead:PINHD-1X3
- added V5, V6, V7, V8: 74161N, 74ttl-din:74161N
- added V9: 7420N, 74ttl-din:7420N
Connections:
- removed net N$29: IC1.I/O2, IC4A.D2
- new net 16B_1: JP2.1, V81.A
- new net 16B_10: JP2.10, V61.B
- new net 16B_11: JP2.11, V61.C
- new net 16B_12: JP2.12, V61.D
- new net 16B_13: JP2.13, V51.A
- new net 16B_14: JP2.14, V51.B
- new net 16B_15: JP2.15, V51.C
- new net 16B_16: JP2.16, V51.D
- new net 16B_2: JP2.2, V81.B
- new net 16B_3: JP2.3, V81.C
- new net 16B_4: JP2.4, V81.D
- new net 16B_5: JP2.5, V71.A
- new net 16B_6: JP2.6, V71.B
- new net 16B_7: JP2.7, V71.C
- new net 16B_8: JP2.8, V71.D
- new net 16B_9: JP2.9, V61.A
- new net 8B_1: IC9A.B1, JP1.1
- new net 8B_2: IC9A.B2, JP1.2
- new net 8B_3: IC9A.B3, JP1.3
- new net 8B_4: IC9A.B4, JP1.4
- new net 8B_5: IC9A.B5, JP1.5
- new net 8B_6: IC9A.B6, JP1.6
- new net 8B_7: IC9A.B7, JP1.7
- new net 8B_8: IC9A.B8, JP1.8
- new net CLK: JP5.1, V51.CLK, V61.CLK, V71.CLK, V81.CLK
- new net CONTROL: IC1.!WE, IC10A.I, IC7A.G, IC8A.G, IC9A.G, JP6.1
- new net COUNT: JP6.2, V51.ENP, V51.ENT, V61.ENP, V61.ENT, V71.ENP, V71.ENT, V81.ENP, V81.ENT
- new net N$40: IC1.A4, IC5A.A5, IC7A.A5
- new net N$41: IC6A.B7, V21.QC, V4/2.A
- new net N$42: IC1.A5, IC5A.A6, IC7A.A6
- new net N$43: IC1.A6, IC5A.A7, IC7A.A7
- new net N$45: IC1.A7, IC5A.A8, IC7A.A8
- new net N$46: IC1.A8, IC6A.A1, IC8A.A1
- new net N$47: IC1.A9, IC6A.A2, IC8A.A2
- new net N$48: IC1.A10, IC6A.A3, IC8A.A3
- new net N$49: IC1.A11, IC6A.A4, IC8A.A4
- new net N$50: IC1.A12, IC6A.A5, IC8A.A5
- new net N$51: IC1.A13, IC6A.A6, IC8A.A6
- new net N$52: IC1.A14, IC6A.A7, IC8A.A7
- new net N$53: IC8A.B7, V51.QC, V9/2.A
- new net N$54: IC8A.B8, V51.QD, V9/2.B, V9/2.C, V9/2.D
- new net N$55: IC7A.B1, V81.QA
- new net N$56: IC7A.B2, V81.QB
- new net N$57: IC7A.B3, V81.QC
- new net N$58: IC7A.B4, V81.QD
- new net N$59: IC7A.B5, V71.QA
- new net N$60: IC7A.B6, V71.QB
- new net N$61: IC7A.B7, V71.QC
- new net N$62: IC7A.B8, V71.QD
- new net N$63: IC8A.B1, V61.QA
- new net N$64: IC8A.B6, V51.QB
- new net N$65: IC8A.B5, V51.QA
- new net N$66: IC8A.B4, V61.QD
- new net N$67: IC8A.B3, V61.QC
- new net N$68: IC8A.B2, V61.QB
- new net N$69: J1.10
- new net N$70: J1.5
- new net N$71: IC1.I/O7, IC4A.D7, IC9A.A8
- new net N$72: IC1.I/O5, IC4A.D5, IC9A.A6
- new net N$73: IC1.I/O6, IC4A.D6, IC9A.A7
- new net N$74: IC1.I/O4, IC4A.D4, IC9A.A5
- new net N$75: IC1.I/O3, IC4A.D3, IC9A.A4
- new net N$76: IC1.I/O2, IC4A.D2, IC9A.A3
- new net N$77: IC1.I/O1, IC4A.D1, IC9A.A2
- new net N$78: IC1.I/O0, IC4A.D0, IC9A.A1
- new net N$79: J1.11
- new net N$8: IC5A.B1, V31.QA
- new net N$80: J1.12
- new net N$81: J1.13
- new net N$82: J1.14
- new net N$83: J1.15
- new net N$9: IC5A.B2, V31.QB
- new net PC_LE: JP6.3, V51.!LOAD, V61.!LOAD, V71.!LOAD, V81.!LOAD
- new net |CLR: V51.!CLR, V61.!CLR, V71.!CLR, V81.!CLR, V9/2.Y
- new net |CONTROL: IC1.!OE, IC10A.O, IC4A.G, IC5A.G, IC6A.G
- net GND: now also IC1.!CS, IC5A.DIR, IC6A.DIR, IC7A.DIR, IC8A.DIR, IC9A.DIR
- net N$10: now also IC5A.B5; no longer IC1.A4
- net N$11: now also IC5A.B7; no longer IC1.A6
- net N$12: now also IC6A.B4; no longer IC1.A11
- net N$13: now also IC5A.B8; no longer IC1.A7
- net N$15: now also IC1.A0, IC5A.A1, IC7A.A1; no longer IC1.A14, V21.QC, V4/2.A
- net N$17: now also IC6A.B1; no longer IC1.A8
- net N$18: now also IC6A.B2; no longer IC1.A9
- net N$19: now also IC6A.B5; no longer IC1.A12
- net N$20: now also IC6A.B6; no longer IC1.A13
- net N$21: now also IC6A.B3; no longer IC1.A5
- net N$26: now also IC5A.B3, V31.QC; no longer IC4A.G, V11.QD
- net N$27: now also J1.6; no longer IC1.I/O0, IC4A.D0
- net N$28: now also J1.1; no longer IC1.I/O1, IC4A.D1
- net N$30: now also J1.2; no longer IC1.I/O3, IC4A.D3
- net N$31: now also J1.8; no longer IC1.I/O4, IC4A.D4
- net N$32: now also J1.3; no longer IC1.I/O5, IC4A.D5
- net N$33: now also J1.9; no longer IC1.I/O6, IC4A.D6
- net N$34: now also J1.4; no longer IC1.I/O7, IC4A.D7
- net N$35: now also IC5A.B4, V31.QD; no longer IC1.A0, V31.QA
- net N$36: now also IC5A.A2, IC7A.A2; no longer V31.QB
- net N$37: now also IC5A.A3, IC7A.A3; no longer V31.QC
- net N$38: now also IC5A.A4, IC7A.A4; no longer V31.QD
- net N$44: now also IC5A.B6; no longer IC1.A10
Other:
- moved on the sheet: IC1, JP1

Commit message: Organized
Parts:
- added LED1, LED2: (no value), led:LED5MM
- added R3, R4: (no value), rcl:R-EU_0204/7
- added R5, R6: (no value), resistor:R-EU_0204/7
- added T1: BC337, transistor:BC337
- J1: SPICEPREFIX (none) -> X
Connections:
- removed net N$30: J1.2
- removed net N$31: J1.8
- removed net N$32: J1.3
- removed net N$33: J1.9
- removed net N$34: J1.4
- removed net N$69: J1.10
- removed net N$70: J1.5
- removed net N$79: J1.11
- removed net N$80: J1.12
- removed net N$81: J1.13
- removed net N$82: J1.14
- removed net N$83: J1.15
- new net D_SIGNAL: IC4A.Y, R5.2
- new net N$29: LED1.C, R4.2
- new net SIGNAL: J1.1, J1.2, J1.3, R6.1, T1.E
- net GND: now also J1.10, J1.5, J1.6, J1.7, J1.8, R3.1, R4.1, R6.2
- net HSYNC: now also J1.13, LED2.A
- net N$27: now also R5.1, T1.B; no longer J1.6
- net N$28: now also LED2.C, R3.2; no longer J1.1
- net VCC: now also T1.C
- net VSYNC: now also J1.14, LED1.A
Other:
- moved on the sheet: C2, IC10A, IC2D, IC2E, J1, JP4, Q1, R1, R2

Commit message: Visual Improvments
Parts:
- J1: value (none) -> DDNM; device Wurth_Elektronik_Electromechanic_Input-Output_Connectors_rev19a:618015325223 -> untitled:DDNM
Other:
- moved on the sheet: J1
Changed lines of the file:
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@@
 <grid distance="0.1" unitdist="inch" unit="inch" style="lines" multiple="1" display="no" altdistance="0.01" altunitdist="inch" altunit="inch"/>
 <layers>
-<layer number="1" name="Top" color="4" fill="1" visible="yes" active="no"/>
-<layer number="2" name="Route2" color="16" fill="1" visible="yes" active="no"/>
-<layer number="3" name="Route3" color="17" fill="1" visible="yes" active="no"/>
-<layer number="4" name="Route4" color="18" fill="1" visible="yes" active="no"/>
-<layer number="5" name="Route5" color="19" fill="1" visible="yes" active="no"/>
-<layer number="6" name="Route6" color="25" fill="1" visible="yes" active="no"/>
-<layer number="7" name="Route7" color="26" fill="1" visible="yes" active="no"/>
-<layer number="8" name="Route8" color="27" fill="1" visible="yes" active="no"/>
-<layer number="9" name="Route9" color="28" fill="1" visible="yes" active="no"/>
-<layer number="10" name="Route10" color="29" fill="1" visible="yes" active="no"/>
-<layer number="11" name="Route11" color="30" fill="1" visible="yes" active="no"/>
-<layer number="12" name="Route12" color="20" fill="1" visible="yes" active="no"/>
-<layer number="13" name="Route13" color="21" fill="1" visible="yes" active="no"/>
-<layer number="14" name="Route14" color="22" fill="1" visible="yes" active="no"/>
-<layer number="15" name="Route15" color="23" fill="1" visible="yes" active="no"/>
-<layer number="16" name="Bottom" color="1" fill="1" visible="yes" active="no"/>
-<layer number="17" name="Pads" color="2" fill="1" visible="yes" active="no"/>
-<layer number="18" name="Vias" color="2" fill="1" visible="yes" active="no"/>
-<layer number="19" name="Unrouted" color="6" fill="1" visible="yes" active="no"/>
-<layer number="20" name="Dimension" color="24" fill="1" visible="yes" active="no"/>
-<layer number="21" name="tPlace" color="7" fill="1" visible="yes" active="no"/>
-<layer number="22" name="bPlace" color="7" fill="1" visible="yes" active="no"/>
-<layer number="23" name="tOrigins" color="15" fill="1" visible="yes" active="no"/>
-<layer number="24" name="bOrigins" color="15" fill="1" visible="yes" active="no"/>
-<layer number="25" name="tNames" color="7" fill="1" visible="yes" active="no"/>
-<layer number="26" name="bNames" color="7" fill="1" visible="yes" active="no"/>
-<layer number="27" name="tValues" color="7" fill="1" visible="yes" active="no"/>
-<layer number="28" name="bValues" color="7" fill="1" visible="yes" active="no"/>
+<layer number="1" name="Top" color="4" fill="1" visible="no" active="no"/>
+<layer number="2" name="Route2" color="16" fill="1" visible="no" active="no"/>
+<layer number="3" name="Route3" color="17" fill="1" visible="no" active="no"/>
+<layer number="4" name="Route4" color="18" fill="1" visible="no" active="no"/>
+<layer number="5" name="Route5" color="19" fill="1" visible="no" active="no"/>
+<layer number="6" name="Route6" color="25" fill="1" visible="no" active="no"/>
+<layer number="7" name="Route7" color="26" fill="1" visible="no" active="no"/>
+<layer number="8" name="Route8" color="27" fill="1" visible="no" active="no"/>
+<layer number="9" name="Route9" color="28" fill="1" visible="no" active="no"/>
+<layer number="10" name="Route10" color="29" fill="1" visible="no" active="no"/>
+<layer number="11" name="Route11" color="30" fill="1" visible="no" active="no"/>
+<layer number="12" name="Route12" color="20" fill="1" visible="no" active="no"/>
+<layer number="13" name="Route13" color="21" fill="1" visible="no" active="no"/>
+<layer number="14" name="Route14" color="22" fill="1" visible="no" active="no"/>
+<layer number="15" name="Route15" color="23" fill="1" visible="no" active="no"/>
+<layer number="16" name="Bottom" color="1" fill="1" visible="no" active="no"/>
+<layer number="17" name="Pads" color="2" fill="1" visible="no" active="no"/>
+<layer number="18" name="Vias" color="2" fill="1" visible="no" active="no"/>
+<layer number="19" name="Unrouted" color="6" fill="1" visible="no" active="no"/>
+<layer number="20" name="Dimension" color="24" fill="1" visible="no" active="no"/>
+<layer number="21" name="tPlace" color="7" fill="1" visible="no" active="no"/>
+<layer number="22" name="bPlace" color="7" fill="1" visible="no" active="no"/>
+<layer number="23" name="tOrigins" color="15" fill="1" visible="no" active="no"/>
+<layer number="24" name="bOrigins" color="15" fill="1" visible="no" active="no"/>
+<layer number="25" name="tNames" color="7" fill="1" visible="no" active="no"/>
+<layer number="26" name="bNames" color="7" fill="1" visible="no" active="no"/>
+<layer number="27" name="tValues" color="7" fill="1" visible="no" active="no"/>
+<layer number="28" name="bValues" color="7" fill="1" visible="no" active="no"/>
 <layer number="29" name="tStop" color="7" fill="3" visible="no" active="no"/>
 <layer number="30" name="bStop" color="7" fill="6" visible="no" active="no"/>
@@
 <layer number="35" name="tGlue" color="7" fill="4" visible="no" active="no"/>
 <layer number="36" name="bGlue" color="7" fill="5" visible="no" active="no"/>
-<layer number="37" name="tTest" color="7" fill="1" visible="yes" active="no"/>
-<layer number="38" name="bTest" color="7" fill="1" visible="yes" active="no"/>
+<layer number="37" name="tTest" color="7" fill="1" visible="no" active="no"/>
+<layer number="38" name="bTest" color="7" fill="1" visible="no" active="no"/>
 <layer number="39" name="tKeepout" color="4" fill="11" visible="no" active="no"/>
 <layer number="40" name="bKeepout" color="1" fill="11" visible="no" active="no"/>
@@
 <layer number="44" name="Drills" color="7" fill="1" visible="no" active="no"/>
 <layer number="45" name="Holes" color="7" fill="1" visible="no" active="no"/>
-<layer number="46" name="Milling" color="3" fill="1" visible="yes" active="no"/>
-<layer number="47" name="Measures" color="7" fill="1" visible="yes" active="no"/>
-<layer number="48" name="Document" color="7" fill="1" visible="yes" active="no"/>
-<layer number="49" name="Reference" color="7" fill="1" visible="yes" active="no"/>
-<layer number="50" name="dxf" color="7" fill="1" visible="yes" active="no"/>
-<layer number="51" name="tDocu" color="7" fill="1" visible="yes" active="no"/>
-<layer number="52" name="bDocu" color="7" fill="1" visible="yes" active="no"/>
-<layer number="53" name="tGND_GNDA" color="7" fill="9" visible="yes" active="no"/>
-<layer number="54" name="bGND_GNDA" color="1" fill="9" visible="yes" active="no"/>
-<layer number="56" name="wert" color="7" fill="1" visible="yes" active="no"/>
-<layer number="57" name="tCAD" color="7" fill="1" visible="yes" active="no"/>
-<layer number="59" name="tCarbon" color="7" fill="1" visible="yes" active="no"/>
-<layer number="60" name="bCarbon" color="7" fill="1" visible="yes" active="no"/>
+<layer number="46" name="Milling" color="3" fill="1" visible="no" active="no"/>
+<layer number="47" name="Measures" color="7" fill="1" visible="no" active="no"/>
+<layer number="48" name="Document" color="7" fill="1" visible="no" active="no"/>
+<layer number="49" name="Reference" color="7" fill="1" visible="no" active="no"/>
+<layer number="50" name="dxf" color="7" fill="1" visible="no" active="no"/>
+<layer number="51" name="tDocu" color="7" fill="1" visible="no" active="no"/>
+<layer number="52" name="bDocu" color="7" fill="1" visible="no" active="no"/>
+<layer number="53" name="tGND_GNDA" color="7" fill="9" visible="no" active="no"/>
+<layer number="54" name="bGND_GNDA" color="1" fill="9" visible="no" active="no"/>
+<layer number="56" name="wert" color="7" fill="1" visible="no" active="no"/>
+<layer number="57" name="tCAD" color="7" fill="1" visible="no" active="no"/>
+<layer number="59" name="tCarbon" color="7" fill="1" visible="no" active="no"/>
+<layer number="60" name="bCarbon" color="7" fill="1" visible="no" active="no"/>
 <layer number="88" name="SimResults" color="9" fill="1" visible="yes" active="yes"/>
 <layer number="89" name="SimProbes" color="9" fill="1" visible="yes" active="yes"/>
@@
 <part name="IC9" library="74xx-eu" library_urn="urn:adsk.eagle:library:85" deviceset="74*245" device="N" package3d_urn="urn:adsk.eagle:package:16429/2" technology="AC"/>
 <part name="IC10" library="74xx-eu" library_urn="urn:adsk.eagle:library:85" deviceset="74*04" device="N" package3d_urn="urn:adsk.eagle:package:16407/2" technology="AC"/>
-<part name="J1" library="Wurth_Elektronik_Electromechanic_Input-Output_Connectors_rev19a" library_urn="urn:adsk.eagle:library:488835" deviceset="618015325223" device="" package3d_urn="urn:adsk.eagle:package:3360028/3">
+<part name="J1" library="untitled" library_urn="urn:adsk.eagle:library:12106798" deviceset="DDNM" device="" package3d_urn="urn:adsk.eagle:package:12106801/4">
 <attribute name="SPICEPREFIX" value="X"/>
 </part>

Commit message: Microcode Added and Ram Updated
Connections:
- removed net PC_LE: JP6.3, V51.!LOAD, V61.!LOAD, V71.!LOAD, V81.!LOAD
- net 16B_16: now also V51.!LOAD, V61.!LOAD, V71.!LOAD, V81.!LOAD; no longer V51.D
Changed lines of the file:
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@@
-</segment>
-</net>
-<net name="PC_LE" class="0">
-<segment>
-<pinref part="V5" gate="1" pin="!LOAD"/>
-<wire x1="284.48" y1="-276.86" x2="284.48" y2="-284.48" width="0.1524" layer="91"/>
-<label x="284.48" y="-284.48" size="1.778" layer="95" rot="R180"/>
-</segment>
-<segment>
-<pinref part="V6" gate="1" pin="!LOAD"/>
-<wire x1="223.52" y1="-276.86" x2="223.52" y2="-284.48" width="0.1524" layer="91"/>
-<label x="223.52" y="-284.48" size="1.778" layer="95" rot="R180"/>
-</segment>
-<segment>
-<pinref part="V7" gate="1" pin="!LOAD"/>
-<wire x1="162.56" y1="-276.86" x2="162.56" y2="-284.48" width="0.1524" layer="91"/>
-<label x="162.56" y="-284.48" size="1.778" layer="95" rot="R180"/>
-</segment>
-<segment>
-<pinref part="V8" gate="1" pin="!LOAD"/>
-<wire x1="101.6" y1="-276.86" x2="101.6" y2="-284.48" width="0.1524" layer="91"/>
-<label x="101.6" y="-287.02" size="1.778" layer="95" rot="R180"/>
-</segment>
-<segment>
-<pinref part="JP6" gate="A" pin="3"/>
-<wire x1="-35.56" y1="-63.5" x2="-30.48" y2="-63.5" width="0.1524" layer="91"/>
-<label x="-30.48" y="-63.5" size="1.778" layer="95"/>
 </segment>
 </net>
@@
 </segment>
 <segment>
-<pinref part="V5" gate="1" pin="D"/>
-<wire x1="327.66" y1="-276.86" x2="327.66" y2="-284.48" width="0.1524" layer="91"/>
-<label x="327.66" y="-284.48" size="1.778" layer="95" rot="MR270"/>
-</segment>
-</net>
+<pinref part="V5" gate="1" pin="!LOAD"/>
+<wire x1="284.48" y1="-276.86" x2="284.48" y2="-284.48" width="0.1524" layer="91"/>
+<label x="284.48" y="-284.48" size="1.778" layer="95" rot="R180"/>
+</segment>
+<segment>
+<pinref part="V6" gate="1" pin="!LOAD"/>
+<wire x1="223.52" y1="-276.86" x2="223.52" y2="-284.48" width="0.1524" layer="91"/>
+<label x="223.52" y="-284.48" size="1.778" layer="95" rot="R180"/>
+</segment>
+<segment>
+<pinref part="V7" gate="1" pin="!LOAD"/>
+<wire x1="162.56" y1="-276.86" x2="162.56" y2="-284.48" width="0.1524" layer="91"/>
+<label x="162.56" y="-284.48" size="1.778" layer="95" rot="R180"/>
+</segment>
+<segment>
+<pinref part="V8" gate="1" pin="!LOAD"/>
+<wire x1="101.6" y1="-276.86" x2="101.6" y2="-284.48" width="0.1524" layer="91"/>
+<label x="101.6" y="-287.02" size="1.778" layer="95" rot="R180"/>
+</segment>
+</net>
