File: Schematics/Main_BoardV2_Divided/proto.sch (EAGLE design)
At the start: 42 parts

Commit message: Microcode Added and Ram Updated
Parts:
- added JP1: (no value), pinhead:PINHD-1X1
Connections:
- new net NNOW2: JP1.1
Changed lines of the file:
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@@
 <pinref part="V2" gate="1" pin="!LOAD"/>
 <wire x1="114.3" y1="83.82" x2="114.3" y2="91.44" width="0.1524" layer="91"/>
-<label x="114.3" y="91.44" size="1.778" layer="95"/>
+<label x="114.3" y="93.98" size="1.778" layer="95"/>
 </segment>
 <segment>
@@
 <port name="|RAM_WRITE" side="right" coord="-12.7" direction="io"/>
 <port name="VCC" side="top" coord="-2.54" direction="io"/>
+<port name="NNOW2" side="right" coord="-17.78" direction="io"/>
 </ports>
 <variantdefs>
@@
 <label x="-259.08" y="58.42" size="1.778" layer="95" rot="R180"/>
 </segment>
-<segment>
-<wire x1="-58.42" y1="111.76" x2="-60.96" y2="111.76" width="0.1524" layer="91"/>
-<label x="-63.5" y="111.76" size="1.778" layer="95" rot="R180"/>
-<pinref part="IC15" gate="A" pin="!A!/B"/>
-<wire x1="-60.96" y1="111.76" x2="-63.5" y2="111.76" width="0.1524" layer="91"/>
-<junction x="-60.96" y="111.76"/>
-</segment>
-<segment>
-<pinref part="IC16" gate="A" pin="!A!/B"/>
-<wire x1="-60.96" y1="71.12" x2="-63.5" y2="71.12" width="0.1524" layer="91"/>
-<label x="-63.5" y="71.12" size="1.778" layer="95" rot="R180"/>
-</segment>
-<segment>
-<pinref part="IC17" gate="A" pin="!A!/B"/>
-<wire x1="-60.96" y1="25.4" x2="-63.5" y2="25.4" width="0.1524" layer="91"/>
-<label x="-63.5" y="25.4" size="1.778" layer="95" rot="R180"/>
-</segment>
-<segment>
-<pinref part="IC18" gate="A" pin="!A!/B"/>
-<wire x1="-60.96" y1="-17.78" x2="-63.5" y2="-17.78" width="0.1524" layer="91"/>
-<label x="-63.5" y="-17.78" size="1.778" layer="95" rot="R180"/>
-</segment>
 </net>
 <net name="8B_8" class="0">
@@
 </segment>
 </net>
+<net name="NNOW2" class="0">
+<segment>
+<wire x1="-58.42" y1="111.76" x2="-60.96" y2="111.76" width="0.1524" layer="91"/>
+<label x="-63.5" y="111.76" size="1.778" layer="95" rot="R180"/>
+<pinref part="IC15" gate="A" pin="!A!/B"/>
+<wire x1="-60.96" y1="111.76" x2="-63.5" y2="111.76" width="0.1524" layer="91"/>
+<junction x="-60.96" y="111.76"/>
+</segment>
+<segment>
+<pinref part="IC16" gate="A" pin="!A!/B"/>
+<wire x1="-60.96" y1="71.12" x2="-63.5" y2="71.12" width="0.1524" layer="91"/>
+<label x="-63.5" y="71.12" size="1.778" layer="95" rot="R180"/>
+</segment>
+<segment>
+<pinref part="IC17" gate="A" pin="!A!/B"/>
+<wire x1="-60.96" y1="25.4" x2="-63.5" y2="25.4" width="0.1524" layer="91"/>
+<label x="-63.5" y="25.4" size="1.778" layer="95" rot="R180"/>
+</segment>
+<segment>
+<pinref part="IC18" gate="A" pin="!A!/B"/>
+<wire x1="-60.96" y1="-17.78" x2="-63.5" y2="-17.78" width="0.1524" layer="91"/>
+<label x="-63.5" y="-17.78" size="1.778" layer="95" rot="R180"/>
+</segment>
+</net>
 </nets>
 </sheet>
@@
 <part name="JP22" library="pinhead" library_urn="urn:adsk.eagle:library:325" deviceset="PINHD-1X2" device="" package3d_urn="urn:adsk.eagle:package:22435/2"/>
 <part name="SV23" library="con-lstb" library_urn="urn:adsk.eagle:library:162" deviceset="MA08-2" device="" package3d_urn="urn:adsk.eagle:package:8335/1"/>
+<part name="JP1" library="pinhead" library_urn="urn:adsk.eagle:library:325" deviceset="PINHD-1X1" device="" package3d_urn="urn:adsk.eagle:package:22485/2"/>
 </parts>
 <sheets>
@@
 <attribute name="NAME" x="267.97" y="51.562" size="1.778" layer="95"/>
 </instance>
+<instance part="JP1" gate="G$1" x="38.1" y="25.4" smashed="yes">
+<attribute name="NAME" x="29.21" y="31.115" size="1.778" layer="95"/>
+<attribute name="VALUE" x="31.75" y="20.32" size="1.778" layer="96"/>
+</instance>
 </instances>
 <busses>
@@
 </segment>
 </net>
+<net name="NNOW2" class="0">
+<segment>
+<portref moduleinst="RAM1" port="NNOW2"/>
+<wire x1="17.78" y1="27.94" x2="27.94" y2="27.94" width="0.1524" layer="91"/>
+<wire x1="27.94" y1="27.94" x2="27.94" y2="25.4" width="0.1524" layer="91"/>
+<pinref part="JP1" gate="G$1" pin="1"/>
+<wire x1="27.94" y1="25.4" x2="35.56" y2="25.4" width="0.1524" layer="91"/>
+<label x="22.86" y="27.94" size="1.778" layer="95"/>
+</segment>
+</net>
